Commit message: Update Fielder WebSocket bridge and ROS2 packages

File: src/axbot_description/urdf/axbot.urdf (robot description, URDF)
Before this commit: robot axbot, 4 links, 3 joints
Links:
- added link base_scan, mass 0.5; visual cylinder length=0.05 radius=0.05
- link laser_frame: geometry 
Joints:
- removed joint laser_joint
- added joint laser_frame_joint: type fixed, parent base_scan, child laser_frame, origin xyz=0 0 0 rpy=0 0 0
- added joint scan_joint: type fixed, parent base_link, child base_scan, origin xyz=0.2 0 0.1 rpy=0 0 0
